File: Microcontroller/PCB/modular-main.sch (EAGLE design)
At the start: 16 parts, among them IC1 7805T, X1 SSW-115-02-G-S

Commit message: Added MARKII PCB designs
Parts:
- removed D1: SSW-115-02-G-S, con-samtec:SSW-115-02-G-S
- added X3: GND, con-samtec:SSW-101-02-G-S
- added X4: VDD, con-samtec:SSW-101-02-G-S
- X1: value SSW-115-02-G-S -> D1; device con-samtec:SSW-115-02-G-S -> con-samtec:SSW-101-02-G-S
Connections:
- net GND: now also X3.1; no longer X1-14.1
- net N$1: now also X1.1; no longer D1-2.1
- net N$28: now also X4.1; no longer X1-15.1
Other:
- moved on the sheet: X1
Changed lines of the file:
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@@
 </classes>
 <parts>
-<part name="X1" library="con-samtec" library_urn="urn:adsk.eagle:library:184" deviceset="SSW-115-02-G-S" device="" value=""/>
-<part name="D1" library="con-samtec" library_urn="urn:adsk.eagle:library:184" deviceset="SSW-115-02-G-S" device="" value=""/>
-<part name="GND8" library="supply1" library_urn="urn:adsk.eagle:library:371" deviceset="GND" device=""/>
 <part name="SUPPLY9" library="supply2" library_urn="urn:adsk.eagle:library:372" deviceset="+5V" device="" value="VDD"/>
 <part name="GND9" library="supply1" library_urn="urn:adsk.eagle:library:371" deviceset="GND" device=""/>
@@
 <part name="+12V1" library="wirepad" library_urn="urn:adsk.eagle:library:412" deviceset="SMD5" device="" package3d_urn="urn:adsk.eagle:package:30841/1"/>
 <part name="GND3" library="wirepad" library_urn="urn:adsk.eagle:library:412" deviceset="SMD5" device="" package3d_urn="urn:adsk.eagle:package:30841/1"/>
+<part name="X3" library="con-samtec" library_urn="urn:adsk.eagle:library:184" deviceset="SSW-101-02-G-S" device="" value="GND"/>
+<part name="X4" library="con-samtec" library_urn="urn:adsk.eagle:library:184" deviceset="SSW-101-02-G-S" device="" value="VDD"/>
+<part name="GND2" library="supply1" library_urn="urn:adsk.eagle:library:371" deviceset="GND" device=""/>
+<part name="X1" library="con-samtec" library_urn="urn:adsk.eagle:library:184" deviceset="SSW-101-02-G-S" device="" value="D1"/>
 </parts>
 <sheets>
@@
 </plain>
 <instances>
-<instance part="X1" gate="-1" x="20.32" y="80.01" smashed="yes">
-<attribute name="VALUE" x="17.78" y="82.55" size="1.778" layer="96"/>
-<attribute name="NAME" x="17.272" y="80.772" size="1.524" layer="95" rot="R180"/>
-</instance>
-<instance part="X1" gate="-2" x="20.32" y="77.47" smashed="yes">
-<attribute name="NAME" x="17.272" y="78.232" size="1.524" layer="95" rot="R180"/>
-</instance>
-<instance part="X1" gate="-3" x="20.32" y="74.93" smashed="yes">
-<attribute name="NAME" x="17.272" y="75.692" size="1.524" layer="95" rot="R180"/>
-</instance>
-<instance part="X1" gate="-4" x="20.32" y="72.39" smashed="yes">
-<attribute name="NAME" x="17.272" y="73.152" size="1.524" layer="95" rot="R180"/>
-</instance>
-<instance part="X1" gate="-5" x="20.32" y="69.85" smashed="yes">
-<attribute name="NAME" x="17.272" y="70.612" size="1.524" layer="95" rot="R180"/>
-</instance>
-<instance part="X1" gate="-6" x="20.32" y="67.31" smashed="yes">
-<attribute name="NAME" x="17.272" y="68.072" size="1.524" layer="95" rot="R180"/>
-</instance>
-<instance part="X1" gate="-7" x="20.32" y="64.77" smashed="yes">
-<attribute name="NAME" x="17.272" y="65.532" size="1.524" layer="95" rot="R180"/>
-</instance>
-<instance part="X1" gate="-8" x="20.32" y="62.23" smashed="yes">
-<attribute name="NAME" x="17.272" y="62.992" size="1.524" layer="95" rot="R180"/>
-</instance>
-<instance part="X1" gate="-9" x="20.32" y="59.69" smashed="yes">
-<attribute name="NAME" x="17.272" y="60.452" size="1.524" layer="95" rot="R180"/>
-</instance>
-<instance part="X1" gate="-10" x="20.32" y="57.15" smashed="yes">
-<attribute name="NAME" x="17.272" y="57.912" size="1.524" layer="95" rot="R180"/>
-</instance>
-<instance part="X1" gate="-11" x="20.32" y="54.61" smashed="yes">
-<attribute name="NAME" x="17.272" y="55.372" size="1.524" layer="95" rot="R180"/>
-</instance>
-<instance part="X1" gate="-12" x="20.32" y="52.07" smashed="yes">
-<attribute name="NAME" x="17.272" y="52.832" size="1.524" layer="95" rot="R180"/>
-</instance>
-<instance part="X1" gate="-13" x="20.32" y="49.53" smashed="yes">
-<attribute name="NAME" x="17.272" y="50.292" size="1.524" layer="95" rot="R180"/>
-</instance>
-<instance part="X1" gate="-14" x="20.32" y="46.99" smashed="yes">
-<attribute name="NAME" x="17.272" y="47.752" size="1.524" layer="95" rot="R180"/>
-</instance>
-<instance part="X1" gate="-15" x="20.32" y="44.45" smashed="yes">
-<attribute name="NAME" x="17.272" y="45.212" size="1.524" layer="95" rot="R180"/>
-</instance>
-<instance part="D1" gate="-1" x="40.64" y="80.01" smashed="yes">
-<attribute name="VALUE" x="38.1" y="82.55" size="1.778" layer="96"/>
-<attribute name="NAME" x="37.592" y="80.772" size="1.524" layer="95" rot="R180"/>
-</instance>
-<instance part="D1" gate="-2" x="40.64" y="77.47" smashed="yes">
-<attribute name="NAME" x="37.592" y="78.232" size="1.524" layer="95" rot="R180"/>
-</instance>
-<instance part="D1" gate="-3" x="40.64" y="74.93" smashed="yes">
-<attribute name="NAME" x="37.592" y="75.692" size="1.524" layer="95" rot="R180"/>
-</instance>
-<instance part="D1" gate="-4" x="40.64" y="72.39" smashed="yes">
-<attribute name="NAME" x="37.592" y="73.152" size="1.524" layer="95" rot="R180"/>
-</instance>
-<instance part="D1" gate="-5" x="40.64" y="69.85" smashed="yes">
-<attribute name="NAME" x="37.592" y="70.612" size="1.524" layer="95" rot="R180"/>
-</instance>
-<instance part="D1" gate="-6" x="40.64" y="67.31" smashed="yes">
-<attribute name="NAME" x="37.592" y="68.072" size="1.524" layer="95" rot="R180"/>
-</instance>
-<instance part="D1" gate="-7" x="40.64" y="64.77" smashed="yes">
-<attribute name="NAME" x="37.592" y="65.532" size="1.524" layer="95" rot="R180"/>
-</instance>
-<instance part="D1" gate="-8" x="40.64" y="62.23" smashed="yes">
-<attribute name="NAME" x="37.592" y="62.992" size="1.524" layer="95" rot="R180"/>
-</instance>
-<instance part="D1" gate="-9" x="40.64" y="59.69" smashed="yes">
-<attribute name="NAME" x="37.592" y="60.452" size="1.524" layer="95" rot="R180"/>
-</instance>
-<instance part="D1" gate="-10" x="40.64" y="57.15" smashed="yes">
-<attribute name="NAME" x="37.592" y="57.912" size="1.524" layer="95" rot="R180"/>
-</instance>
-<instance part="D1" gate="-11" x="40.64" y="54.61" smashed="yes">
-<attribute name="NAME" x="37.592" y="55.372" size="1.524" layer="95" rot="R180"/>
-</instance>
-<instance part="D1" gate="-12" x="40.64" y="52.07" smashed="yes">
-<attribute name="NAME" x="37.592" y="52.832" size="1.524" layer="95" rot="R180"/>
-</instance>
-<instance part="D1" gate="-13" x="40.64" y="49.53" smashed="yes">
-<attribute name="NAME" x="37.592" y="50.292" size="1.524" layer="95" rot="R180"/>
-</instance>
-<instance part="D1" gate="-14" x="40.64" y="46.99" smashed="yes">
-<attribute name="NAME" x="37.592" y="47.752" size="1.524" layer="95" rot="R180"/>
-</instance>
-<instance part="D1" gate="-15" x="40.64" y="44.45" smashed="yes">
-<attribute name="NAME" x="37.592" y="45.212" size="1.524" layer="95" rot="R180"/>
-</instance>
-<instance part="GND8" gate="1" x="25.4" y="46.99" smashed="yes" rot="R90">
-<attribute name="VALUE" x="27.94" y="44.45" size="1.778" layer="96" rot="R90"/>
-</instance>
 <instance part="SUPPLY9" gate="+5V" x="64.77" y="114.3" smashed="yes">
 <attribute name="VALUE" x="62.865" y="117.475" size="1.778" layer="96"/>
@@
 <attribute name="NAME" x="52.6542" y="95.123" size="1.778" layer="95" rot="R270"/>
 <attribute name="VALUE" x="47.498" y="95.123" size="1.778" layer="96" rot="R270"/>
+</instance>
+<instance part="X3" gate="-1" x="20.32" y="55.88" smashed="yes">
+<attribute name="VALUE" x="17.78" y="58.42" size="1.778" layer="96"/>
+<attribute name="NAME" x="17.272" y="56.642" size="1.524" layer="95" rot="R180"/>
+</instance>
+<instance part="X4" gate="-1" x="20.32" y="50.8" smashed="yes">
+<attribute name="VALUE" x="17.78" y="53.34" size="1.778" layer="96"/>
+<attribute name="NAME" x="17.272" y="51.562" size="1.524" layer="95" rot="R180"/>
+</instance>
+<instance part="GND2" gate="1" x="43.18" y="53.34" smashed="yes">
+<attribute name="VALUE" x="40.64" y="50.8" size="1.778" layer="96"/>
+</instance>
+<instance part="X1" gate="-1" x="39.878" y="77.47" smashed="yes">
+<attribute name="VALUE" x="37.338" y="80.01" size="1.778" layer="96"/>
+<attribute name="NAME" x="36.83" y="78.232" size="1.524" layer="95" rot="R180"/>
 </instance>
 </instances>
@@
 <nets>
 <net name="GND" class="0">
-<segment>
-<pinref part="X1" gate="-14" pin="1"/>
-<pinref part="GND8" gate="1" pin="GND"/>
-</segment>
 <segment>
 <pinref part="IC1" gate="A1" pin="GND"/>
@@
 <wire x1="50.8" y1="88.9" x2="48.26" y2="88.9" width="0.1524" layer="91"/>
 <junction x="48.26" y="88.9"/>
+</segment>
+<segment>
+<pinref part="X3" gate="-1" pin="1"/>
+<pinref part="GND2" gate="1" pin="GND"/>
+<wire x1="43.18" y1="55.88" x2="22.86" y2="55.88" width="0.1524" layer="91"/>
 </segment>
 </net>
@@
 <pinref part="R7" gate="G$1" pin="1"/>
 <wire x1="44.45" y1="111.76" x2="43.18" y2="111.76" width="0.1524" layer="91"/>
-<pinref part="X1" gate="-15" pin="1"/>
 <wire x1="43.18" y1="111.76" x2="41.91" y2="111.76" width="0.1524" layer="91"/>
-<wire x1="22.86" y1="44.45" x2="22.86" y2="38.1" width="0.1524" layer="91"/>
+<wire x1="22.86" y1="44.45" x2="22.86" y2="43.18" width="0.1524" layer="91"/>
+<wire x1="22.86" y1="43.18" x2="22.86" y2="38.1" width="0.1524" layer="91"/>
 <wire x1="22.86" y1="38.1" x2="5.08" y2="38.1" width="0.1524" layer="91"/>
 <wire x1="5.08" y1="38.1" x2="5.08" y2="121.92" width="0.1524" layer="91"/>
@@
 <wire x1="43.18" y1="121.92" x2="43.18" y2="111.76" width="0.1524" layer="91"/>
 <junction x="43.18" y="111.76"/>
+<pinref part="X4" gate="-1" pin="1"/>
+<wire x1="22.86" y1="50.8" x2="22.86" y2="44.45" width="0.1524" layer="91"/>
 </segment>
 </net>
 <net name="N$1" class="0">
 <segment>
-<pinref part="D1" gate="-2" pin="1"/>
-<wire x1="43.18" y1="77.47" x2="49.53" y2="77.47" width="0.1524" layer="91"/>
+<wire x1="43.18" y1="77.47" x2="42.418" y2="77.47" width="0.1524" layer="91"/>
+<wire x1="42.418" y1="77.47" x2="49.53" y2="77.47" width="0.1524" layer="91"/>
 <wire x1="49.53" y1="77.47" x2="49.53" y2="35.56" width="0.1524" layer="91"/>
 <wire x1="49.53" y1="35.56" x2="104.14" y2="35.56" width="0.1524" layer="91"/>
@@
 <pinref part="0" gate="G$1" pin="DIN"/>
 <wire x1="104.14" y1="59.69" x2="93.98" y2="59.69" width="0.1524" layer="91"/>
-</segment>
-</net>
+<pinref part="X1" gate="-1" pin="1"/>
+<junction x="42.418" y="77.47"/>
+</segment>
+</net>
